Commit message: Ya se probo con datos de lidar no simulados
Ahora tocara probar con datos de LIDAR fisicos

File: install/basic_mobile_robot/share/basic_mobile_robot/models/basic_mobile_bot_v2.urdf (robot description, URDF)
Before this commit: robot basic_mobile_bot, 6 links, 5 joints
Links:
- removed link lidar_link
- added link laser, mass 0.114; collision cylinder length=0.18 radius=0.0508; visual cylinder length=0.18 radius=0.0508
Joints:
- joint lidar_joint: child lidar_link -> laser

Commit message: Ya se finalizo el SLAM Simulado
Ahora falta probar el SLAM FISICO

File: install/basic_mobile_robot/share/basic_mobile_robot/models/basic_mobile_bot_v2.urdf (robot description, URDF)
Before this commit: robot basic_mobile_bot, 6 links, 5 joints
Links:
- removed link laser
- added link lidar_link, mass 0.114; collision cylinder length=0.18 radius=0.0508; visual cylinder length=0.18 radius=0.0508
Joints:
- joint lidar_joint: child laser -> lidar_link
